Commit message: trying move_base plugin

File: description/chassis.xacro (robot description, xacro)
@@ -11,5 +11,5 @@
     </inertial>
     <visual>
-      <origin xyz="0 0 0" rpy="1.57079632679 0 0"/>
+      <origin xyz="0 0 0.12" rpy="1.57079632679 0 0"/>
       <geometry>
         <mesh filename="package://ratf_description/meshes/base_link.stl" scale="0.001 0.001 0.001"/>
@@ -18,5 +18,5 @@
     </visual>
     <collision>
-      <origin xyz="0 0 0" rpy="1.57079632679 0 0"/>
+      <origin xyz="0 0 0.12" rpy="1.57079632679 0 0"/>
       <geometry>
         <mesh filename="package://ratf_description/meshes/base_link.stl" scale="0.001 0.001 0.001"/>

File: description/ratf5dpo.urdf.xacro (robot description, xacro)
@@ -2,3 +2,12 @@
 <robot xmlns:xacro="http://www.ros.org/wiki/xacro"  name="ratf_description">
     <xacro:include filename="chassis.xacro" />
+    <plugin name="gazebo_ros_planar_move" filename="libgazebo_ros_planar_move.so">
+        <robotNamespace>/robot_namespace</robotNamespace>
+        <commandTopic>cmd_vel</commandTopic>
+        <odometryTopic>odom</odometryTopic>
+        <odometryFrame>odom</odometryFrame>
+        <robotBaseFrame>base_link</robotBaseFrame>
+        <odometryRate>20.0</odometryRate>
+        <cmdTimeout>-1</cmdTimeout>
+    </plugin>
 </robot>
